File: dinosat/dinosat.kicad_sch (KiCad schematic)
At the start: 28 parts, among them J1 USB_C_Receptacle_USB2.0_16P, J2 Conn_01x02, Q1 FS8205A, U1 STM32U5A5ZJTx, U2 TP4056-42-ESOP8, U3 DW01A, U4 TPS63060

Commit message: Lots of schematic work
Parts:
- added C10, C12, C13, C14, C15, C16, C17, C18, C20, C22, C23, C24, C27, C8, C9: 100nF, Capacitor_SMD:C_0603_1608Metric, symbol Device:C
- added C11, C25: 4.7uF, Capacitor_SMD:C_0603_1608Metric, symbol Device:C
- added C19: 10uF, Capacitor_SMD:C_0603_1608Metric, symbol Device:C
- added C21, C26: 1uF, Capacitor_SMD:C_0603_1608Metric, symbol Device:C
- added C28: 0.1uF, Capacitor_SMD:C_0603_1608Metric, symbol Device:C
- added J3: Conn_02x05_Odd_Even, Connector_PinHeader_1.27mm:PinHeader_2x05_P1.27mm_Vertical, symbol Connector_Generic:Conn_02x05_Odd_Even
- added R11: 10K, Resistor_SMD:R_0603_1608Metric, symbol Device:R
- added SW1, SW2: SW_Push, Button_Switch_SMD:SW_SPST_TL3342, symbol Switch:SW_Push
- C1, C2, C3, C4, C5, C6, C7: footprint (none) -> Capacitor_SMD:C_0603_1608Metric
- D1: footprint (none) -> Diode_SMD:D_SMA
- D2, D3: footprint (none) -> LED_SMD:LED_0603_1608Metric
- J1: footprint (none) -> Connector_USB:USB_C_Receptacle_GCT_USB4105-xx-A_16P_TopMnt_Horizontal
- J2: value Conn_01x02 -> Battery JST; footprint (none) -> Connector_JST:JST_PH_B2B-PH-K_1x02_P2.00mm_Vertical
- L1: footprint (none) -> Inductor_SMD:L_0603_1608Metric
- R1, R10, R2, R3, R4, R5, R6, R7, R8, R9: footprint (none) -> Resistor_SMD:R_0603_1608Metric
Connections:
- net +3V3: now also U1.131 (VDDIO2), U1.6 (VBAT), U1.95 (VDDIO2), C10.2, C12.1, C13.1, C14.1, C15.1, C16.1, C17.1, C18.1, C19.1, C20.1, C21.1, C22.1, C23.1, C24.1, C25.1, C8.1, C9.1, J3.1 (Pin_1), SW2.1
- net GND: now also C10.1, C11.1, C12.2, C13.2, C14.2, C15.2, C16.2, C17.2, C18.2, C19.2, C20.2, C21.2, C22.2, C23.2, C24.2, C25.2, C28.1, C8.2, C9.2, J3.3 (Pin_3), J3.5 (Pin_5), J3.7 (Pin_7), J3.9 (Pin_9), R11.1, SW1.1
- net D+: now reaches J1.A6 (D+)
- net D+: now also J1.B6 (D+)
- net D-: now reaches J1.A7 (D-)
- net D-: now also J1.B7 (D-)
- net SWDIO: now reaches U1.105 (PA13)
- net SWDIO: now also J3.2 (Pin_2)
- net SWCLK: now reaches U1.109 (PA14)
- net SWCLK: now also J3.4 (Pin_4)
- net JTDI: now reaches U1.110 (PA15)
- net JTDI: now also J3.8 (Pin_8)
- net at U1.138 (PH3): now also R11.2, SW2.2
- net NRST: now reaches U1.25 (NRST)
- net NRST: now also C28.2, J3.10 (Pin_10), SW1.2
- net at U1.70 (VCAP): now also C11.2
- new net: C26.1, C27.1
- new net: C26.2, C27.2
Other:
- note added: "STM32U5A5"
- note added: "Specifies Charge Current"
- moved on the sheet: U1
