File: dinosat/dinosat.kicad_sch (KiCad schematic)
At the start: 53 parts, among them J1 USB_C_Receptacle_USB2.0_16P, J2 Battery JST, J3 Conn_02x05_Odd_Even, Q1 FS8205A, SW1 SW_Push, SW2 SW_Push, U1 STM32U5A5ZJTx, U2 TP4056-42-ESOP8, U3 DW01A, U4 TPS63060

Commit message: Rah
Parts:
- added C29, C32: 100nF, Capacitor_SMD:C_0402_1005Metric, symbol Device:C
- added C30, C31: 10uF, Capacitor_SMD:C_0603_1608Metric, symbol Device:C
- added C33: 10pF, symbol Device:C
- added R12: 220, symbol Device:R
- added U5: LR1121IMLTRT, LR1121IMLTRT:QFN50P500X500X100-33N, symbol LR1121IMLTRT:LR1121IMLTRT
- added Y1: TCXO-14, Oscillator:Oscillator_DIP-14, symbol Oscillator:TCXO-14
Connections:
- net +3V3: now also C29.1, C30.1, C31.2, C32.2, U5.15 (VBAT), U5.2 (VBAT_RF)
- net GND: now also C29.2, C30.2, C31.1, C32.1, U5.13 (GND), U5.33 (GND), Y1.7 (GND)
- net RFBUSY: now reaches U1.100 (PA8)
- net RFBUSY: now also U5.25 (DIO0/BUSY)
- net IRQ: now reaches U1.101 (PA9)
- net IRQ: now also U5.9 (DIO9)
- net SCK: now reaches U1.35 (PA1)
- net SCK: now also U5.23 (DIO2)
- net NSS: now reaches U1.40 (PA4)
- net NSS: now also U5.24 (DIO1)
- net NRESET: now reaches U1.41 (PA5)
- net NRESET: now also U5.6 (~{RESET})
- net MISO: now reaches U1.42 (PA6)
- net MISO: now also U5.21 (DIO4)
- net MOSI: now reaches U1.43 (PA7)
- net MOSI: now also U5.22 (DIO3)
- new net: C33.2, R12.1
- new net: R12.2, Y1.8 (OUT)
- new net: U5.16 (DNC), U5.17 (DNC), U5.18 (DNC), U5.27 (DNC), U5.28 (DNC)
- new net: U5.3 (VTCXO), Y1.14 (Vcc)
- new net: C33.1, U5.4 (XTA)
Other:
- note added: "LoRa"
- note added: "ST Link"

Commit message: IO, usb
Parts:
- added C34, C35: 10uF, Capacitor_SMD:C_0603_1608Metric, symbol Device:C
- added C36: 0.1uF, Capacitor_SMD:C_0603_1608Metric, symbol Device:C
- added C37: 10pF, Capacitor_SMD:C_0603_1608Metric, symbol Device:C
- added J4: SolarPanel JST, Connector_JST:JST_PH_B2B-PH-K_1x02_P2.00mm_Vertical, symbol Connector_Generic:Conn_01x02
- added J5: Conn_01x15, Connector_PinHeader_1.27mm:PinHeader_1x15_P1.27mm_Vertical, symbol Connector_Generic:Conn_01x15
- added J6, J7: Conn_01x16, Connector_PinHeader_1.27mm:PinHeader_1x16_P1.27mm_Vertical, symbol Connector_Generic:Conn_01x16
- added J8, J9: Conn_01x10, Connector_PinHeader_1.27mm:PinHeader_1x10_P1.27mm_Vertical, symbol Connector_Generic:Conn_01x10
- added L2: 1uH, Inductor_SMD:L_0603_1608Metric, symbol Device:L
- added R13: 900K, Resistor_SMD:R_0603_1608Metric, symbol Device:R
- added R14: 100K, Resistor_SMD:R_0603_1608Metric, symbol Device:R
- added R15: 1M, Resistor_SMD:R_0603_1608Metric, symbol Device:R
- added U6: TPS63060, Package_SON:Texas_S-PWSON-N10_ThermalVias, symbol Regulator_Switching:TPS63060
- C33: footprint (none) -> Capacitor_SMD:C_0603_1608Metric
- R12: footprint (none) -> Resistor_SMD:R_0603_1608Metric
Connections:
- net +3V3: now also J8.1 (Pin_1), J8.2 (Pin_2), J8.3 (Pin_3), J8.4 (Pin_4), J8.5 (Pin_5), J9.1 (Pin_1), J9.2 (Pin_2), J9.3 (Pin_3), J9.4 (Pin_4), J9.5 (Pin_5)
- net D+: now also U1.104 (PA12)
- net D-: now also U1.103 (PA11)
- net GND: now also C34.2, C35.2, C36.2, C37.2, J4.1 (Pin_1), J8.10 (Pin_10), J8.6 (Pin_6), J8.7 (Pin_7), J8.8 (Pin_8), J8.9 (Pin_9), J9.10 (Pin_10), J9.6 (Pin_6), J9.7 (Pin_7), J9.8 (Pin_8), J9.9 (Pin_9), R14.2, U6.11 (PGND), U6.4 (PS/SYNC), U6.7 (GND)
- net PG: now also R15.2, U6.5 (PG)
- net VIN+: now also R13.1, R15.1, U6.9 (VOUT)
- net PC10: now reaches U1.111 (PC10)
- net PC10: now also J6.11 (Pin_11)
- net PC11: now reaches U1.112 (PC11)
- net PC11: now also J6.12 (Pin_12)
- net PC12: now reaches U1.113 (PC12)
- net PC12: now also J6.13 (Pin_13)
- net PD0: now reaches U1.114 (PD0)
- net PD0: now also J7.1 (Pin_1)
- net PD1: now reaches U1.115 (PD1)
- net PD1: now also J7.2 (Pin_2)
- net PD2: now reaches U1.116 (PD2)
- net PD2: now also J7.3 (Pin_3)
- net PD3: now reaches U1.117 (PD3)
- net PD3: now also J7.4 (Pin_4)
- net PD4: now reaches U1.118 (PD4)
- net PD4: now also J7.5 (Pin_5)
- net PD5: now reaches U1.119 (PD5)
- net PD5: now also J7.6 (Pin_6)
- net PD6: now reaches U1.122 (PD6)
- net PD6: now also J7.7 (Pin_7)
- net PD7: now reaches U1.123 (PD7)
- net PD7: now also J7.8 (Pin_8)
- net PB3: now reaches U1.133 (PB3)
- net PB3: now also J5.4 (Pin_4)
- net PB4: now reaches U1.134 (PB4)
- net PB4: now also J5.5 (Pin_5)
- net PB5: now reaches U1.135 (PB5)
- net PB5: now also J5.6 (Pin_6)
- net PB6: now reaches U1.136 (PB6)
- net PB6: now also J5.7 (Pin_7)
- net PB7: now reaches U1.137 (PB7)
- net PB7: now also J5.8 (Pin_8)
- net PB8: now reaches U1.139 (PB8)
- net PB8: now also J5.9 (Pin_9)
- net PB9: now reaches U1.140 (PB9)
- net PB9: now also J5.10 (Pin_10)
- net PC0: now reaches U1.26 (PC0)
- net PC0: now also J6.1 (Pin_1)
- net PC1: now reaches U1.27 (PC1)
- net PC1: now also J6.2 (Pin_2)
- net PC2: now reaches U1.28 (PC2)
- net PC2: now also J6.3 (Pin_3)
- net PC3: now reaches U1.29 (PC3)
- net PC3: now also J6.4 (Pin_4)
- net PC4: now reaches U1.44 (PC4)
- net PC4: now also J6.5 (Pin_5)
- net PC5: now reaches U1.45 (PC5)
- net PC5: now also J6.6 (Pin_6)
- net PB0: now reaches U1.46 (PB0)
- net PB0: now also J5.1 (Pin_1)
- net PB1: now reaches U1.47 (PB1)
- net PB1: now also J5.2 (Pin_2)
- net PB2: now reaches U1.48 (PB2)
- net PB2: now also J5.3 (Pin_3)
- net PB10: now reaches U1.69 (PB10)
- net PB10: now also J5.11 (Pin_11)
- net PC13: now reaches U1.7 (PC13)
- net PC13: now also J6.14 (Pin_14)
- net PB12: now reaches U1.73 (PB12)
- net PB12: now also J5.12 (Pin_12)
- net PB13: now reaches U1.74 (PB13)
- net PB13: now also J5.13 (Pin_13)
- net PB14: now reaches U1.75 (PB14)
- net PB14: now also J5.14 (Pin_14)
- net PB15: now reaches U1.76 (PB15)
- net PB15: now also J5.15 (Pin_15)
- net PD8: now reaches U1.77 (PD8)
- net PD8: now also J7.9 (Pin_9)
- net PD9: now reaches U1.78 (PD9)
- net PD9: now also J7.10 (Pin_10)
- net PD10: now reaches U1.79 (PD10)
- net PD10: now also J7.11 (Pin_11)
- net PC14: now reaches U1.8 (PC14)
- net PC14: now also J6.15 (Pin_15)
- net PD11: now reaches U1.80 (PD11)
- net PD11: now also J7.12 (Pin_12)
- net PD12: now reaches U1.81 (PD12)
- net PD12: now also J7.13 (Pin_13)
- net PD13: now reaches U1.82 (PD13)
- net PD13: now also J7.14 (Pin_14)
- net PD14: now reaches U1.85 (PD14)
- net PD14: now also J7.15 (Pin_15)
- net PD15: now reaches U1.86 (PD15)
- net PD15: now also J7.16 (Pin_16)
- net PC15: now reaches U1.9 (PC15)
- net PC15: now also J6.16 (Pin_16)
- net PC6: now reaches U1.96 (PC6)
- net PC6: now also J6.7 (Pin_7)
- net PC7: now reaches U1.97 (PC7)
- net PC7: now also J6.8 (Pin_8)
- net PC8: now reaches U1.98 (PC8)
- net PC8: now also J6.9 (Pin_9)
- net PC9: now reaches U1.99 (PC9)
- net PC9: now also J6.10 (Pin_10)
- net RFBUSY renamed NBUSY
- new net: L2.2, U6.1 (L1)
- new net: L2.1, U6.10 (L2)
- new net: C36.1, U6.6 (VAUX)
- new net: C37.1, R13.2, R14.1, U6.8 (FB)
- new net PANELIN+: C34.1, C35.1, J4.2 (Pin_2), U6.2 (VIN), U6.3 (EN)
Other:
- note added: "SPI + LoRa"
- note added: "STM32 IO"
- note added: "Solar Panel Managment"
- note added: "USB"
